File: kicad/singingcard.kicad_pcb (KiCad board)
At the start: 2 copper layers, 85 x 55 mm, 16 parts, among them J1 Speaker 8ohm, J2 Pull-Tab, SW1 Button, U1 ISD3900FYI, U2 W25Q16JVSSIQ

Commit message: Complete schematic/ERC/DRC workflow and generate fab files
- Fixed schematic generator to use correct footprint names
- Created local symbol and footprint libraries
- ERC: 12 warnings (library config), 0 errors
- DRC: 26 warnings (cosmetic), 0 errors, 0 unconnected
- PCB fully routed with 188 tracks and vias
- Generated Gerber, drill, and position files for JLCPCB
- Created JLCPCB-ready zip file
- Updated skill file with ERC/DRC severity guidance
- Added final renders for visual inspection

🤖 Generated with [Claude Code](https://claude.com/claude-code)

Co-Authored-By: Claude <noreply@anthropic.com>
Parts:
- moved U2 7.00 mm to (166.0, 119.5)
- moved BT1 5.00 mm to (167.0, 127.5)
Routing:
- net GND: track 0.00 -> 179.0 mm, vias 0 -> 3
- net +3V: track 0.00 -> 176.4 mm
- net GPIO1_BTN: track 0.00 -> 52.7 mm, vias 0 -> 2
- net N$1: track 0.00 -> 52.0 mm, vias 0 -> 2
- net N$2: track 0.00 -> 49.8 mm, vias 0 -> 2
- net SPI_SCK: track 0.00 -> 35.4 mm, vias 0 -> 2
- net GPIO2_TAB: track 0.00 -> 34.8 mm, vias 0 -> 2
- net SPI_MOSI: track 0.00 -> 33.4 mm
- net GPIO0_LDR: track 0.00 -> 33.1 mm
- net SPI_MISO: track 0.00 -> 27.1 mm
- net SPI_CS: track 0.00 -> 24.5 mm
- net RESET: track 0.00 -> 20.7 mm, vias 0 -> 2
- net VREG: track 0.00 -> 19.4 mm, vias 0 -> 2
- net CSB: track 0.00 -> 15.4 mm
